Commit message: Adding Hokuyo features :
hokuyo could now be used as kinect with :
export TURTLEBOT_3D_SENSOR=kinect
   OR
export TURTLEBOT_3D_SENSOR=hokuyo

File: turtlebot_description/urdf/sensors/hokuyo.urdf.xacro (robot description, xacro)
@@ -1,31 +1,31 @@
 <?xml version="1.0"?>
 <robot name="sensor_hokuyo" xmlns:xacro="http://ros.org/wiki/xacro">
- <xacro:include filename="$(find turtlebot_description)/urdf/turtlebot_gazebo.urdf.xacro"/>
- <xacro:include filename="$(find turtlebot_description)/urdf/turtlebot_properties.urdf.xacro"/>
- <xacro:macro name="sensor_hokuyo" params="parent">
-     <link name="laser_joint">
-   <collision>
-     <origin xyz="0 0 0" rpy="0 0 0"/>
-     <geometry>
+  <xacro:include filename="$(find turtlebot_description)/urdf/turtlebot_gazebo.urdf.xacro"/>
+  <xacro:include filename="$(find turtlebot_description)/urdf/turtlebot_properties.urdf.xacro"/>
+  <xacro:macro name="sensor_hokuyo" params="parent">
+  <joint name="hokuyo_joint" type="fixed">
+    <origin xyz="-0.005 0.00 0.360" rpy="3.14159 0 0" />
+    <parent link="${parent}"/>
+    <child link="hokuyo_frame"/>
+  </joint>
+  <link name="hokuyo_frame">
+    <visual>
+      <origin xyz="0 0 0" rpy="0 0 0"/>
+      <geometry>
+        <mesh filename="package://turtlebot_description/meshes/sensors/hokuyo.dae"/>
+      </geometry>
+    </visual>
+    <collision>
+      <origin xyz="0 0 0" rpy="0 0 0"/>
+      <geometry>
         <box size="0.1 0.1 0.1"/>
-     </geometry>
-   </collision>
-   <visual>
-     <origin xyz="0 0 0" rpy="0 0 0"/>
-     <geometry>
-       <mesh filename="package://turtlebot_description/meshes/sensors/hokuyo.dae"/>
-     </geometry>
-   </visual>
-   <inertial>
-     <mass value="1e-5" />
-     <origin xyz="0 0 0" rpy="0 0 0"/>
-     <inertia ixx="1e-6" ixy="0" ixz="0" iyy="1e-6" iyz="0" izz="1e-6" />
-   </inertial>
- </link>
- <joint name="hokuyo_joint" type="fixed">
-   <origin xyz="-0.005 0.00 0.360" rpy="3.14159 0 0" />
-   <parent link="${parent}"/>
-   <child link="laser"/>
- </joint>
- </xacro:macro>
+      </geometry>
+    </collision>
+    <inertial>
+      <mass value="1e-5" />
+      <origin xyz="0 0 0" rpy="0 0 0"/>
+      <inertia ixx="1e-6" ixy="0" ixz="0" iyy="1e-6" iyz="0" izz="1e-6" />
+    </inertial>
+  </link>
+  </xacro:macro>
 </robot>

Commit message: Adding conditional hokuyo support

File: turtlebot_description/urdf/sensors/hokuyo.urdf.xacro (robot description, xacro)
@@ -4,10 +4,10 @@
   <xacro:include filename="$(find turtlebot_description)/urdf/turtlebot_properties.urdf.xacro"/>
   <xacro:macro name="sensor_hokuyo" params="parent">
-  <joint name="hokuyo_joint" type="fixed">
+  <joint name="laser" type="fixed">
     <origin xyz="-0.005 0.00 0.360" rpy="3.14159 0 0" />
-    <parent link="${parent}"/>
-    <child link="hokuyo_frame"/>
+    <parent link="base_link"/>
+    <child link="base_laser_link"/>
   </joint>
-  <link name="hokuyo_frame">
+  <link name="base_laser_link">
     <visual>
       <origin xyz="0 0 0" rpy="0 0 0"/>

File: turtlebot_description/urdf/turtlebot_library.urdf.xacro (robot description, xacro)
@@ -19,5 +19,5 @@
   <xacro:include filename="$(find turtlebot_description)/urdf/sensors/astra.urdf.xacro"/>
   <xacro:include filename="$(find turtlebot_description)/urdf/sensors/r200.urdf.xacro"/>
-  <xacro:include filename="$(find turtlebot_description)/urdf/sensors/hokuyo.urdf.xacro"/>
+<!--  <xacro:include filename="$(find turtlebot_description)/urdf/sensors/hokuyo.urdf.xacro"/> -->
 <!-- avant merge pour astra, la ligne dessus (urdf hokuyo) était comentée et pas le bloc suivant. C'est l'un ou l'autre-->
 <!--
